Commit message: Aded actuators to gazebo, it can be controlled via ros_msgs, z_axis have joint position, wheels have velocity control

File: urdf/include/gazebo_control.xacro (robot description, xacro)
@@ -1,21 +1,8 @@
 <?xml version="1.0"?>
 <robot xmlns:xacro="http://www.ros.org/wiki/xacro">
-    <gazebo>
-        <plugin name="diff_drive" filename="libgazebo_ros_diff_drive.so">
-            <!-- Wheel Information -->
-            <left_joint>left_wheel_joint</left_joint>
-            <right_joint>right_wheel_joint</right_joint>
-            <wheel_separation>0.35</wheel_separation>
-            <wheel_diameter>0.1</wheel_diameter>
-            <!-- Limits -->
-            <max_wheel_torque>200</max_wheel_torque>
-            <max_wheel_acceleration>10.0</max_wheel_acceleration>
-            <!-- Output -->
-            <odometry_frame>odom</odometry_frame>
-            <robot_base_frame>base_link</robot_base_frame>
-            <publish_odom>true</publish_odom>
-            <publish_odom_tf>true</publish_odom_tf>
-            <publish_wheel_tf>true</publish_wheel_tf>
-        </plugin>
-    </gazebo>
+  <gazebo>
+    <plugin name="gazebo_ros_control" filename="libgazebo_ros_control.so">
+      <robotNamespace>/farmbeast</robotNamespace>
+    </plugin>
+  </gazebo>
 </robot>

File: urdf/robot.urdf.xacro (robot description, xacro)
@@ -61,5 +61,5 @@
         <collision>
             <geometry>
-                <cylinder radius="0.02" length="0.06"/>
+               <cylinder radius="0.03" length="0.1"/>
             </geometry>
         </collision>
@@ -68,4 +68,13 @@
         </xacro:inertial_cylinder>
     </link>
+    <transmission name="left_front_z_axis_trans">
+      <type>transmission_interface/SimpleTransmission</type>
+      <joint name="left_front_z_axis_joint">
+        <hardwareInterface>hardware_interface/PositionJointInterface</hardwareInterface>
+      </joint>
+      <actuator name="left_front_z_axis_actuator">
+        <mechanicalReduction>1</mechanicalReduction>
+      </actuator>
+    </transmission>
     <!-- left front wheel -->
     <joint name="left_front_wheel_joint" type="continuous">
@@ -84,5 +93,5 @@
         <collision>
             <geometry>
-                <cylinder radius="0.05" length="0.04"/>
+                <cylinder radius="0.1" length="0.04"/>
             </geometry>
         </collision>
@@ -91,4 +100,13 @@
         </xacro:inertial_cylinder>
     </link>
+    <transmission name="left_front_wheel_trans">
+      <type>transmission_interface/SimpleTransmission</type>
+      <joint name="left_front_wheel_joint">
+        <hardwareInterface>hardware_interface/VelocityJointInterface</hardwareInterface>
+      </joint>
+      <actuator name="left_front_wheel_actuator">
+        <mechanicalReduction>1</mechanicalReduction>
+      </actuator>
+    </transmission>
     <gazebo reference="left_wheel">
         <material>Gazebo/Blue</material>
@@ -111,5 +129,5 @@
         <collision>
             <geometry>
-                <cylinder radius="0.02" length="0.06"/>
+               <cylinder radius="0.03" length="0.1"/>
             </geometry>
         </collision>
@@ -118,4 +136,13 @@
         </xacro:inertial_cylinder>
     </link>
+    <transmission name="left_back_z_axis_trans">
+      <type>transmission_interface/SimpleTransmission</type>
+      <joint name="left_back_z_axis_joint">
+        <hardwareInterface>hardware_interface/PositionJointInterface</hardwareInterface>
+      </joint>
+      <actuator name="left_back_z_axis_actuator">
+        <mechanicalReduction>1</mechanicalReduction>
+      </actuator>
+    </transmission>
     <!-- left back wheel -->
     <joint name="left_back_wheel_joint" type="continuous">
@@ -134,5 +161,5 @@
         <collision>
             <geometry>
-                <cylinder radius="0.05" length="0.04"/>
+                <cylinder radius="0.1" length="0.04"/>
             </geometry>
         </collision>
@@ -141,4 +168,13 @@
         </xacro:inertial_cylinder>
     </link>
+    <transmission name="left_back_wheel_trans">
+      <type>transmission_interface/SimpleTransmission</type>
+      <joint name="left_back_wheel_joint">
+        <hardwareInterface>hardware_interface/VelocityJointInterface</hardwareInterface>
+      </joint>
+      <actuator name="left_back_wheel_actuator">
+        <mechanicalReduction>1</mechanicalReduction>
+      </actuator>
+    </transmission>
     <gazebo reference="left_wheel">
         <material>Gazebo/Blue</material>
@@ -161,5 +197,5 @@
         <collision>
             <geometry>
-                <cylinder radius="0.02" length="0.06"/>
+                <cylinder radius="0.03" length="0.1"/>
             </geometry>
         </collision>
@@ -168,4 +204,13 @@
         </xacro:inertial_cylinder>
     </link>
+    <transmission name="right_front_z_axis_trans">
+      <type>transmission_interface/SimpleTransmission</type>
+      <joint name="right_front_z_axis_joint">
+        <hardwareInterface>hardware_interface/PositionJointInterface</hardwareInterface>
+      </joint>
+      <actuator name="right_front_z_axis_actuator">
+        <mechanicalReduction>1</mechanicalReduction>
+      </actuator>
+    </transmission>
     <!-- right front wheel -->
     <joint name="right_front_wheel_joint" type="continuous">
@@ -184,5 +229,5 @@
         <collision>
             <geometry>
-                <cylinder radius="0.05" length="0.04"/>
+               <cylinder radius="0.1" length="0.04"/>
             </geometry>
         </collision>
@@ -191,4 +236,13 @@
         </xacro:inertial_cylinder>
     </link>
+    <transmission name="right_front_wheel_trans">
+      <type>transmission_interface/SimpleTransmission</type>
+      <joint name="right_front_wheel_joint">
+        <hardwareInterface>hardware_interface/VelocityJointInterface</hardwareInterface>
+      </joint>
+      <actuator name="right_front_wheel_actuator">
+        <mechanicalReduction>1</mechanicalReduction>
+      </actuator>
+    </transmission>
     <gazebo reference="right_wheel">
         <material>Gazebo/Blue</material>
@@ -211,5 +265,5 @@
         <collision>
             <geometry>
-                <cylinder radius="0.02" length="0.06"/>
+                <cylinder radius="0.03" length="0.1"/>
             </geometry>
         </collision>
@@ -218,4 +272,13 @@
         </xacro:inertial_cylinder>
     </link>
+    <transmission name="right_back_z_axis_trans">
+      <type>transmission_interface/SimpleTransmission</type>
+      <joint name="right_back_z_axis_joint">
+        <hardwareInterface>hardware_interface/PositionJointInterface</hardwareInterface>
+      </joint>
+      <actuator name="right_back_z_axis_actuator">
+        <mechanicalReduction>1</mechanicalReduction>
+      </actuator>
+    </transmission>
     <!-- right back wheel -->
     <joint name="right_back_wheel_joint" type="continuous">
@@ -234,5 +297,5 @@
         <collision>
             <geometry>
-                <cylinder radius="0.05" length="0.04"/>
+                <cylinder radius="0.1" length="0.04"/>
             </geometry>
         </collision>
@@ -241,6 +304,21 @@
         </xacro:inertial_cylinder>
     </link>
+    <transmission name="right_back_wheel_trans">
+      <type>transmission_interface/SimpleTransmission</type>
+      <joint name="right_back_wheel_joint">
+        <hardwareInterface>hardware_interface/VelocityJointInterface</hardwareInterface>
+      </joint>
+      <actuator name="right_back_wheel_actuator">
+        <mechanicalReduction>1</mechanicalReduction>
+      </actuator>
+    </transmission>
     <gazebo reference="right_wheel">
         <material>Gazebo/Blue</material>
     </gazebo>
+    <!-- ROS cotntroll-->
+    <gazebo>
+        <plugin name="gazebo_ros_control" filename="libgazebo_ros_control.so">
+            <robotNamespace>/farmbeast</robotNamespace>
+        </plugin>
+    </gazebo>
 </robot>
