Commit message: Created a simple control

File: urdf/robot.urdf.xacro (robot description, xacro)
@@ -37,5 +37,5 @@
             </geometry>
         </collision>
-        <xacro:inertial_box mass="1" x="0.5" y="0.5" z="0.3">
+        <xacro:inertial_box mass="2" x="0.5" y="0.5" z="0.3">
             <origin xyz="0 0 0" rpy="0 0 0"/>
         </xacro:inertial_box>
@@ -77,4 +77,7 @@
       </actuator>
     </transmission>
+    <gazebo reference="left_front_z_axis">
+        <material>Gazebo/Orange</material>
+    </gazebo>
     <!-- left front wheel -->
     <joint name="left_front_wheel_joint" type="continuous">
@@ -109,8 +112,10 @@
       </actuator>
     </transmission>
-    <gazebo reference="left_wheel">
+    <gazebo reference="left_front_wheel">
         <material>Gazebo/Blue</material>
-    </gazebo>
-<!-- Left back z axis -->
+        <mu1 value="200"/>
+        <mu2 value="100"/>
+    </gazebo>
+    <!-- Left back z axis -->
     <joint name="left_back_z_axis_joint" type="revolute">
         <parent link="base_link"/>
@@ -145,4 +150,7 @@
       </actuator>
     </transmission>
+    <gazebo reference="left_back_z_axis">
+        <material>Gazebo/Orange</material>
+    </gazebo>
     <!-- left back wheel -->
     <joint name="left_back_wheel_joint" type="continuous">
@@ -177,6 +185,8 @@
       </actuator>
     </transmission>
-    <gazebo reference="left_wheel">
+    <gazebo reference="left_back_wheel">
         <material>Gazebo/Blue</material>
+        <mu1 value="200"/>
+        <mu2 value="100"/>
     </gazebo>
     <!-- right front z axis -->
@@ -213,4 +223,7 @@
       </actuator>
     </transmission>
+    <gazebo reference="right_front_z_axis">
+        <material>Gazebo/Orange</material>
+    </gazebo>
     <!-- right front wheel -->
     <joint name="right_front_wheel_joint" type="continuous">
@@ -245,8 +258,10 @@
       </actuator>
     </transmission>
-    <gazebo reference="right_wheel">
+    <gazebo reference="right_front_wheel">
         <material>Gazebo/Blue</material>
-    </gazebo>
-<!-- right back z axis -->
+        <mu1 value="200"/>
+        <mu2 value="100"/>
+    </gazebo>
+    <!-- right back z axis -->
     <joint name="right_back_z_axis_joint" type="revolute">
         <parent link="base_link"/>
@@ -281,4 +296,7 @@
       </actuator>
     </transmission>
+    <gazebo reference="right_back_z_axis">
+        <material>Gazebo/Orange</material>
+    </gazebo>
     <!-- right back wheel -->
     <joint name="right_back_wheel_joint" type="continuous">
@@ -313,6 +331,8 @@
       </actuator>
     </transmission>
-    <gazebo reference="right_wheel">
+    <gazebo reference="right_back_wheel">
         <material>Gazebo/Blue</material>
+        <mu1 value="200"/>
+        <mu2 value="100"/>
     </gazebo>
     <!-- ROS cotntroll-->
@@ -322,3 +342,12 @@
         </plugin>
     </gazebo>
+    <!--Velodyne include-->
+    <xacro:arg name="gpu" default="false"/>
+    <xacro:property name="gpu" value="$(arg gpu)" />
+    <xacro:arg name="organize_cloud" default="false"/>
+    <xacro:property name="organize_cloud" value="$(arg organize_cloud)" />
+    <xacro:include filename="$(find velodyne_description)/urdf/VLP-16.urdf.xacro"/>
+    <xacro:VLP-16 parent="base_link" name="velodyne" topic="/velodyne_points" organize_cloud="${organize_cloud}" hz="10" samples="440" gpu="${gpu}" min_range="0.1" max_range="10.0" >
+        <origin xyz="0.25 0 0.3" rpy="0 0.5 0" />
+     </xacro:VLP-16>
 </robot>
